File: hardware/v3/introAu.sch (EAGLE design)
At the start: 45 parts, among them Q1 CERAMIC_RESONATOR_SMD6M00G53Z

Commit message: Trying to make this perfect. Too many changes to count.
Parts:
- added D4, D5, D6, D7: (no value), jumper:SJ
Connections:
- removed net A0: JP1.1
- removed net D14: U$2.PB3(MISO)
- removed net D15: U$2.PB1(SCK)
- removed net D16: U$2.PB2(MOSI)
- removed net N$1: R10.1, U$2.PD1(SDA)
- removed net N$2: R2.1, U$2.PC6
- removed net N$3: R9.1, U$2.PD0(SCL)
- removed net N$4: R8.1, U$2.PD4(ADC8)
- new net N$12: D7.2, JP3.1
- new net N$15: D5.2, JP3.3
- new net N$16: D6.2, JP3.2
- new net N$17: D4.2, JP3.4
- net COL1: now also U$2.PB4(ADC11); no longer U$2.PD7(ADC10)
- net COL2: now also U$2.PB5(ADC12); no longer U$2.PE6
- net COL3: now also U$2.PB7; no longer U$2.PB4(ADC11)
- net COL4: now also U$2.PD6(ADC9); no longer U$2.PB5(ADC12)
- net D11: no longer U$2.PB7
- net D12: no longer U$2.PD6(ADC9)
- net D2: now also U$2.PD1(SDA)
- net D3: now also U$2.PD0(SCL)
- net D4: now also D4.1, R10.1, U$2.PD4(ADC8); no longer JP3.4
- net D5: now also D5.1, R9.1, U$2.PC6; no longer JP3.3
- net D6: now also D6.1, R8.1, U$2.PD7(ADC10); no longer JP3.2
- net D7: now also D7.1, R2.1, U$2.PE6; no longer JP3.1
- net MISO: now also U$2.PB3(MISO)
- net MOSI: now also U$2.PB2(MOSI)
- net SCK: now also U$2.PB1(SCK)
Other:
- moved on the sheet: R10, R2, R8, R9

Commit message: Made more critical changes
Parts:
- added C5: 10uF, rcl:C-EUC0805
- added L2: MF-MSMF050-2, EagleLibrary_Wuerth_Elektronik_eiSos_rev15c:WE-CBF_1812(HC)
- Q1: value CERAMIC_RESONATOR_SMD6M00G53Z -> CERAMIC_RESONATOR_SMD; device MESH_Arduino:CERAMIC_RESONATOR_SMD6M00G53Z -> MESH_Arduino:CERAMIC_RESONATOR_SMD
- renumbered U$4 to Z2, U$6 to Z1
Connections:
- new net N$1: L2.1, U$3.+5V
- net +5V: now also C5.1, L2.2, R11.2; no longer S2.3, S2.4, U$3.+5V
- net COL1: now also LED20.A, LED21.A, LED22.A, LED28.A, R10.2; no longer LED23.C, LED27.C, LED28.C, LED4.C, U$2.PB4(ADC11)
- net COL2: now also LED17.A, LED18.A, LED19.A, LED23.A, R9.2; no longer LED17.C, LED22.C, LED24.C, LED9.C, U$2.PB5(ADC12)
- net COL3: now also LED24.A, LED25.A, LED26.A, LED27.A, R8.2; no longer LED10.C, LED18.C, LED21.C, LED25.C, U$2.PB7
- net COL4: now also LED10.A, LED14.A, LED4.A, LED9.A, R2.2; no longer LED14.C, LED19.C, LED20.C, LED26.C, U$2.PD6(ADC9)
- net GND: now also C5.2, S2.2; no longer R11.2
- net RESET: now also S2.3, S2.4; no longer S2.1, S2.2
- net ROW1: now also LED23.C, LED27.C, LED28.C, LED4.C, U$2.PB4(ADC11); no longer LED20.A, LED21.A, LED22.A, LED28.A, R10.2
- net ROW2: now also LED17.C, LED22.C, LED24.C, LED9.C, U$2.PB5(ADC12); no longer LED17.A, LED18.A, LED19.A, LED23.A, R9.2
- net ROW3: now also LED10.C, LED18.C, LED21.C, LED25.C, U$2.PB7; no longer LED24.A, LED25.A, LED26.A, LED27.A, R8.2
- net ROW4: now also LED14.C, LED19.C, LED20.C, LED26.C, U$2.PD6(ADC9); no longer LED10.A, LED14.A, LED4.A, LED9.A, R2.2
Other:
- moved on the sheet: C1, C2, C3, D4, D5, D6, D7, JP1, JP2, JP3, JP4, JP5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
