File: hardware/v3/introAu.brd (EAGLE design)
At the start: 61.5 x 56.4 mm, 46 parts, among them Q1 CERAMIC_RESONATOR_SMD6M00G53Z

Commit message: Trying to make this perfect. Too many changes to count.
Parts:
- added D4, D5, D6, D7: (no value), jumper:SJ
- moved JP5 24.5 mm to (3.05, 33.5)
- moved R11 7.22 mm to (5.33, 7.62)
- moved C3 6.43 mm to (2.03, 23.9), turned to 270 degrees
- moved U$1 4.33 mm to (49.5, 2.29)
- moved S2 4.32 mm to (29.7, 9.14), turned to 90 degrees
- moved R10 3.70 mm to (28.4, 18.0)
- moved R5 2.09 mm to (19.9, 42.8), turned to 0 degrees
- moved L1 1.55 mm to (9.65, 31.5)
- moved C2 1.52 mm to (11.7, 11.4)
- moved R7 1.48 mm to (4.32, 23.9)
- moved U$4 0.99 mm to (9.27, 19.3), turned to 180 degrees
- moved R6 0.92 mm to (6.35, 23.9)
- moved U$6 0.57 mm to (3.05, 19.6)
- moved S1 0.51 mm to (6.22, 40.5)
- moved R9 0.25 mm to (40.6, 11.2)
Connections:
- removed net A0: JP1.1
- removed net D14: U$2.11
- removed net D15: U$2.9
- removed net D16: U$2.10
- removed net N$1: R10.1, U$2.19
- removed net N$2: R2.P$1, U$2.31
- removed net N$3: R9.1, U$2.18
- removed net N$4: R8.1, U$2.25
- new net N$12: D7.2, JP3.1
- new net N$15: D5.2, JP3.3
- new net N$16: D6.2, JP3.2
- new net N$17: D4.2, JP3.4
- net COL1: now also U$2.28; no longer U$2.27
- net COL2: now also U$2.29; no longer U$2.1
- net COL3: now also U$2.12; no longer U$2.28
- net COL4: now also U$2.26; no longer U$2.29
- net D11: no longer U$2.12
- net D12: no longer U$2.26
- net D2: now also U$2.19
- net D3: now also U$2.18
- net D4: now also D4.1, R10.1, U$2.25; no longer JP3.4
- net D5: now also D5.1, R9.1, U$2.31; no longer JP3.3
- net D6: now also D6.1, R8.1, U$2.27; no longer JP3.2
- net D7: now also D7.1, R2.P$1, U$2.1; no longer JP3.1
- net MISO: now also U$2.11
- net MOSI: now also U$2.10
- net SCK: now also U$2.9
Routing:
- net D7: track 0.00 -> 72.7 mm, vias 0 -> 4
- net D5: track 0.00 -> 56.4 mm, vias 0 -> 3
- net N$4: track 54.4 -> 0.00 mm, vias 2 -> 1
- net D6: track 0.00 -> 50.5 mm, vias 0 -> 2
- net D11: track 41.4 -> 0.00 mm, vias 2 -> 0
- net D4: track 0.00 -> 40.8 mm, vias 0 -> 6
- net N$2: track 36.8 -> 0.00 mm
- net ROW3: track 2.26 -> 37.0 mm
- net D12: track 30.3 -> 0.00 mm, vias 2 -> 0
- net D3: track 0.00 -> 29.2 mm, vias 0 -> 2
- net D2: track 0.00 -> 28.1 mm
- net N$3: track 25.9 -> 0.00 mm, vias 0 -> 1
- net RESET: track 92.9 -> 116.1 mm, vias 4 -> 6
- net MISO: track 0.00 -> 21.8 mm, vias 0 -> 1
- net SCK: track 0.00 -> 17.3 mm, vias 0 -> 1
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Other:
- board text added: "+5V"
- board text added: "A1"
- board text added: "A2"
- board text added: "A3"
- board text added: "A4"
- board text added: "A5"
- board text added: "AREF"
- board text added: "BUTTON"
- board text added: "D0"
- board text added: "D1"
- board text added: "D13"
- board text added: "D2"
- board text added: "D3"
- board text added: "D4"
- board text added: "D5"
- board text added: "D6"
- board text added: "D7"
- board text added: "GND"
- board text added: "Hacker Board"
- board text added: "MHacks 6"
- board text added: "NC"
- board text added: "POTENTIO- METER"
- board text added: "RESET"
- board text removed: "10k"
- board text removed: "1k"

Commit message: Made more critical changes
Parts:
- removed U$4, U$6: 3.6V Zener, SparkFun-DiscreteSemi:SOD-323
- added C5: 10uF, rcl:C0805
- added L2: MF-MSMF050-2, EagleLibrary_Wuerth_Elektronik_eiSos_rev15c:WE-CBF_1812(W=7.3)
- added Z1, Z2: 3.6V Zener, SparkFun-DiscreteSemi:SOD-323
- Q1: value CERAMIC_RESONATOR_SMD6M00G53Z -> CERAMIC_RESONATOR_SMD
- moved C1 39.0 mm to (10.9, 19.9)
- moved C2 24.4 mm to (10.7, 35.8), turned to 90 degrees
- moved C3 4.32 mm to (6.35, 23.9)
- moved D7 2.59 mm to (24.4, 10.0)
- moved U$5 2.29 mm to (50.2, 47.8)
- moved R6 2.03 mm to (4.32, 23.9)
- moved R7 2.03 mm to (2.29, 23.9)
- moved D6 1.52 mm to (22.1, 6.86)
- moved C4 1.08 mm to (27.7, 22.4)
- moved S1 1.05 mm to (5.97, 41.5)
- moved D5 1.02 mm to (17.8, 6.86)
- moved R1 0.72 mm to (36.3, 42.2)
- moved PWR 0.57 mm to (36.3, 45.5)
- moved R11 0.25 mm to (5.33, 7.37)
- moved Q1 0.25 mm to (17.0, 14.5)
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Connections:
- new net N$1: L2.1, U$3.P$1
- net +5V: now also C5.1, L2.2, R11.2; no longer S2.3, S2.4, U$3.P$1
- net COL1: now also LED20.A, LED21.A, LED22.A, LED28.A, R10.2; no longer LED23.C, LED27.C, LED28.C, LED4.K, U$2.28
- net COL2: now also LED17.A, LED18.A, LED19.A, LED23.A, R9.2; no longer LED17.C, LED22.C, LED24.C, LED9.K, U$2.29
- net COL3: now also LED24.A, LED25.A, LED26.A, LED27.A, R8.2; no longer LED10.K, LED18.C, LED21.C, LED25.C, U$2.12
- net COL4: now also LED10.A, LED14.A, LED4.A, LED9.A, R2.P$2; no longer LED14.K, LED19.C, LED20.C, LED26.C, U$2.26
- net GND: now also C5.2, S2.2, U$3.P$5, Z1.1, Z2.1; no longer R11.2, U$3.P$4, U$4.1, U$6.1
- net N$7: now also Z1.2; no longer U$6.2
- net N$9: now also Z2.2; no longer U$4.2
- net RESET: now also S2.3, S2.4; no longer S2.1, S2.2
- net ROW1: now also LED23.C, LED27.C, LED28.C, LED4.K, U$2.28; no longer LED20.A, LED21.A, LED22.A, LED28.A, R10.2
- net ROW2: now also LED17.C, LED22.C, LED24.C, LED9.K, U$2.29; no longer LED17.A, LED18.A, LED19.A, LED23.A, R9.2
- net ROW3: now also LED10.K, LED18.C, LED21.C, LED25.C, U$2.12; no longer LED24.A, LED25.A, LED26.A, LED27.A, R8.2
- net ROW4: now also LED14.K, LED19.C, LED20.C, LED26.C, U$2.26; no longer LED10.A, LED14.A, LED4.A, LED9.A, R2.P$2
Routing:
- net COL3: track 59.9 -> 36.3 mm, vias 5 -> 0
- net ROW3: track 37.0 -> 59.9 mm, vias 0 -> 5
- net COL4: track 51.5 -> 30.7 mm, vias 3 -> 0
- net ROW4: track 30.7 -> 51.4 mm, vias 0 -> 3
- net COL2: track 52.9 -> 36.2 mm, vias 3 -> 0
- net COL1: track 59.3 -> 43.3 mm, vias 2 -> 0
- net ROW2: track 37.0 -> 52.8 mm, vias 0 -> 3
- net ROW1: track 44.2 -> 57.6 mm, vias 0 -> 2
- net +5V: track 154.8 -> 162.1 mm, vias 9 -> 10
- net UCAP: track 12.2 -> 6.55 mm, vias 2 -> 0
- net D4: track 40.8 -> 36.7 mm, vias 6 -> 2
- net N$12: track 8.54 -> 11.4 mm
- net D7: track 72.7 -> 69.8 mm
- net N$1: track 0.00 -> 2.69 mm, vias 1 -> 0
- net RD-: track 9.41 -> 11.7 mm
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Other:
- board text added: "C1"
- board text added: "C2"
- board text added: "C3"
- board text added: "C4"
- board text added: "L1"
- board text added: "L2"
- board text added: "R1"
- board text added: "R10"
- board text added: "R11"
- board text added: "R3"
- board text added: "R6"
- board text added: "R7"
- board text added: "R8"
- board text added: "R9"
- board text added: "Z1"
- board text added: "Z2"
- board text removed: "COL2"
- board text removed: "COL3"
- board text removed: "ROW2"
- board text removed: "ROW3"

Commit message: Fiddled with GND polygons
Parts:
- moved C5 0.80 mm to (10.2, 11.7)
- moved Q1 0.57 mm to (17.5, 14.2)
- moved L2 0.25 mm to (11.0, 16.3)
- turned C1 to 180 degrees
Routing:
- net +5V: track 162.1 -> 164.7 mm
- net N$9: track 16.3 -> 17.3 mm
- net AREF: track 68.1 -> 67.3 mm
- net N$7: track 17.4 -> 18.0 mm
- net N$6: track 6.22 -> 6.77 mm
- net D4: track 36.7 -> 37.2 mm
Other:
- board text removed: "L2"
